File: TuringMain/TuringMain.kicad_pcb (KiCad board)
At the start: 2 copper layers, 119 x 95 mm, 102 parts, among them IC1 TL072P, IC2 78L09, IC3 78L09, J1 Conn_01x10_Male, T1 2N3904, U1 TL074_

Commit message: Main Board Updates
Fixed GND errors and flipped expansion headers to back of the board
Parts:
- GATES1, PULSES1: moved to B.Cu
- moved GATES1 2.56 mm to (113.5, 52.7), turned to -90 degrees
- moved PULSES1 2.46 mm to (113.5, 135.3), turned to -90 degrees
Routing:
- net /PULSE2: track 42.6 -> 58.3 mm, vias 1 -> 0
- net /PULSE1: track 117.9 -> 127.0 mm
- net /GATE6: track 31.6 -> 36.8 mm
- net /GATE3: track 31.6 -> 35.5 mm
- net /PULSE8: track 53.4 -> 56.4 mm
- net /PULSE4: track 59.3 -> 62.0 mm
- net /PULSE6: track 41.2 -> 43.7 mm
- net /PULSE5: track 38.7 -> 41.1 mm, vias 0 -> 1
- net /PULSE7: track 43.5 -> 45.8 mm
- net /GATE2: track 29.5 -> 27.4 mm
- net /PULSE3: track 47.7 -> 49.7 mm
- net /GATE1: track 33.5 -> 35.5 mm, vias 1 -> 0
- net /GATE5: track 37.2 -> 39.0 mm
- net /NOISE: track 103.0 -> 101.3 mm
- net /GATE4: track 39.5 -> 38.3 mm
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
Commit message: Manufacturing Updates
Parts:
- C26, C27: moved to B.Cu

Commit message: Manufacturing Updates
Rotary Switch Panel Drill Corrected
Panel Graphics Changed (Name changed from Turing Machine to The Halting Problem)
Updated silkscreen on mainboard with circuit corrections and component values.
Parts:
- moved UNK2 2.55 mm to (60.0, 68.7), turned to -90 degrees
- moved UNK3 2.55 mm to (60.0, 78.7), turned to -90 degrees
- moved UNK4 2.55 mm to (60.0, 88.7), turned to -90 degrees
- moved UNK5 2.55 mm to (60.0, 98.7), turned to -90 degrees
- moved UNK6 2.55 mm to (60.0, 108.7), turned to -90 degrees
- moved UNK7 2.55 mm to (60.0, 118.7), turned to -90 degrees
- moved UNK8 2.55 mm to (60.0, 128.7), turned to -90 degrees
- moved UNK1 2.55 mm to (60.0, 58.7), turned to -90 degrees
- turned PULS1 to -90 degrees
Connections:
- AND_1 pad 7: /GND -> GND
- AND_2 pad 7: /GND -> GND
- BUFFER1 pad 8: /GND -> GND
- BUFFER2 pad 14: /GND -> GND
- BUFFER2 pad 8: /GND -> GND
- C1 pad 2: /GND -> GND
- C13 pad 2: /GND -> GND
- C14 pad 1: /GND -> GND
- C15 pad 1: /GND -> GND
- C16 pad 1: /GND -> GND
- C19 pad 1: /GND -> GND
- C2 pad 2: /GND -> GND
- C20 pad 1: /GND -> GND
- C21 pad 1: /GND -> GND
- C22 pad 1: /GND -> GND
- C23 pad 1: /GND -> GND
- C24 pad 1: /GND -> GND
- C25 pad 1: /GND -> GND
- C26 pad 1: Net-(U$2-Pad13) -> GND
- C27 pad 1: Net-(U$2-Pad3) -> GND
- C3 pad 2: /GND -> GND
- C4 pad 2: /GND -> GND
- C5 pad 2: /GND -> GND
- C6 pad 1: /GND -> GND
- C7 pad 1: /GND -> GND
- C8 pad 2: /GND -> GND
- CLK1 pad 1: /GND -> GND
- GATES1 pad 13: /GND -> GND
- GATES1 pad 14: /GND -> GND
- IC1 pad 3: /GND -> GND
- IC2 pad 2: /GND -> GND
- IC3 pad 2: /GND -> GND
- J1 pad 1: /GND -> GND
- J1 pad 10: /GND -> GND
- PULS1 pad 1: Net-(PULS1-Pad1) -> GND
- PULS1 pad 2: /GND -> Net-(R17-Pad2)
- PULSES1 pad 13: /GND -> GND
- PULSES1 pad 14: /GND -> GND
- R1 pad 2: /GND -> GND
- R10 pad 1: /GND -> GND
- R11 pad 1: /GND -> GND
- R12 pad 2: /GND -> GND
- R14 pad 1: /GND -> GND
- R15 pad 1: /GND -> GND
- R16 pad 1: /GND -> GND
- R17 pad 2: Net-(PULS1-Pad1) -> Net-(R17-Pad2)
- R21 pad 1: /GND -> GND
- R27 pad 1: /GND -> GND
- R4 pad 2: /GND -> GND
- R6 pad 2: /GND -> GND
- R8 pad 2: /GND -> GND
- R9 pad 1: /GND -> GND
- SCALE1 pad 1: /GND -> GND
- SHIFTREG_EXT1 pad 14: /GND -> GND
- SHIFTREG_EXT1 pad 6: /GND -> GND
- SHIFTREG_EXT1 pad 8: /GND -> GND
- SHIFTREG_MAIN1 pad 14: /GND -> GND
- SHIFTREG_MAIN1 pad 6: /GND -> GND
- SHIFTREG_MAIN1 pad 8: /GND -> GND
- SV1 pad 3: /GND -> GND
- SV1 pad 4: /GND -> GND
- SV1 pad 5: /GND -> GND
- SV1 pad 6: /GND -> GND
- SV1 pad 7: /GND -> GND
- SV1 pad 8: /GND -> GND
- SWITCH_IC1 pad 3: /GND -> GND
- SWITCH_IC1 pad 7: /GND -> GND
- SWITCH_IC1 pad 9: /GND -> GND
- T1 pad 2: /GND -> GND
- TL431 pad 2: /GND -> GND
- U$2 pad 1: /GND -> GND
- U$2 pad 13: Net-(U$2-Pad13) -> /+12V
- U$2 pad 2: /GND -> GND
- U$2 pad 3: Net-(U$2-Pad3) -> /-12V
- U1 pad 10: /GND -> GND
- U1 pad 12: /GND -> GND
- U1 pad 3: /GND -> GND
- UNK1 pad 1: /B1 -> Net-(R21-Pad2)
- UNK1 pad 2: Net-(R21-Pad2) -> /B1
- UNK2 pad 1: /B2 -> Net-(R16-Pad2)
- UNK2 pad 2: Net-(R16-Pad2) -> /B2
- UNK3 pad 1: /B3 -> Net-(R15-Pad2)
- UNK3 pad 2: Net-(R15-Pad2) -> /B3
- UNK4 pad 1: /B4 -> Net-(R14-Pad2)
- UNK4 pad 2: Net-(R14-Pad2) -> /B4
- UNK5 pad 1: /B5 -> Net-(R8-Pad1)
- UNK5 pad 2: Net-(R8-Pad1) -> /B5
- UNK6 pad 1: /B6 -> Net-(R6-Pad1)
- UNK6 pad 2: Net-(R6-Pad1) -> /B6
- UNK7 pad 1: /B7 -> Net-(R4-Pad1)
- UNK7 pad 2: Net-(R4-Pad1) -> /B7
- UNK8 pad 1: /B8 -> Net-(R1-Pad1)
- UNK8 pad 2: Net-(R1-Pad1) -> /B8
- WRITE1 pad 3: /GND -> GND
Routing:
- net Net-(U$2-Pad13): track 21.7 -> 0.00 mm
- net /+12V: track 390.9 -> 411.6 mm
- net Net-(R17-Pad2): track 0.00 -> 17.6 mm
- net Net-(PULS1-Pad1): track 17.6 -> 0.00 mm
- net /-12V: track 243.8 -> 259.5 mm
- net Net-(U$2-Pad3): track 10.6 -> 0.00 mm
- net /B3: track 266.5 -> 268.6 mm
- net /B4: track 222.5 -> 223.4 mm
- net /B8: track 171.8 -> 171.3 mm
- net GND: vias 0 -> 7
- net /GND: vias 6 -> 0
- added copper zone on B.Cu, net GND
- added copper zone on F.Cu, net GND
- removed copper zone on B.Cu, net /GND
- removed copper zone on F.Cu, net /GND
Other:
- board text removed: "Music Thing Modular Turing Machine February 2016 CC-BY-SA"

Commit message: Minor Main Board updates
Parts:
- IC2, IC3, TL431: footprint Package_TO_SOT_THT:TO-92_Inline -> ao_tht:TO-92_Inline_Wide
- moved IC2 3.19 mm to (68.1, 52.0), turned to -90 degrees
- moved IC3 2.92 mm to (68.1, 64.9), turned to -90 degrees
- moved TL431 2.67 mm to (160.1, 106.9)
Routing:
- net GND: track 0.00 -> 5.99 mm
- net Net-(BUFFER1-Pad1): track 12.9 -> 9.08 mm
- net Net-(BUFFER2-Pad1): track 13.7 -> 10.3 mm
- net /B3: track 268.6 -> 271.8 mm
- net Net-(R20-Pad2): track 18.2 -> 20.9 mm
- net Net-(C11-Pad1): track 66.3 -> 64.5 mm
- net /GATE5: track 39.0 -> 37.6 mm
- net /+12V: track 411.6 -> 412.8 mm
- net Net-(C24-Pad2): track 93.4 -> 92.4 mm
